Commit message: 並列化のためのファイル整理する準備

File: models/arena_1/arena.urdf (robot description, URDF)
Before this commit: robot arena, 1 links, 0 joints
Links:
- link arena_link: geometry collision mesh filename=package://phers_framework/models/arena_1/arena.dae scale=4.5 4.5 1; visual mesh filename=package://phers_framework/models/arena_1/arena.dae scale=4.5 4.5 1

Commit message: 5m間隔に変更

File: models/arena_1/arena.urdf (robot description, URDF)
Before this commit: robot arena, 1 links, 0 joints
Links:
- link arena_link: geometry collision mesh filename=package://phers_framework/models/arena_1/arena.dae scale=1 1 1; visual mesh filename=package://phers_framework/models/arena_1/arena.dae scale=1 1 1

Commit message: rospy.sleepを導入。また、stdを行動別に設定

File: models/arena_1/arena.urdf (robot description, URDF)
Before this commit: robot arena, 1 links, 0 joints
Links:
- link arena_link: geometry collision mesh filename=package://phers_framework/models/arena_1/arena.dae scale=4 4 1; visual mesh filename=package://phers_framework/models/arena_1/arena.dae scale=4 4 1
